File: pcb/StrangerFamily.kicad_pcb (KiCad board)
At the start: 2 copper layers, 90 x 50 mm, 26 parts, among them J1 LCD_Conn, J2 Power_LEDs, J3 Output_LED, J4 LED_Out2, J5 Raspberry_Pi_zero, J6 LED_Out2, Q2 BSS138, Q3 BSS138, Q4 BSS138, U1 74LVC2T45DC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

Commit message: Update kicad project version
Connections:
- net /Nano_~Reset renamed /Nano_~{Reset}
- net /RPi_Nano_~Reset renamed /RPi_Nano_~{Reset}
Other:
- net class Default removed
- net class Power removed
